File: stm32_page.kicad_sch (KiCad schematic)
At the start: 46 parts, among them J1 PZ254V-11-03P_C2937625, J2 PZ254V-11-03P_C2937625, J5 PZ254V-11-03P_C2937625, SW2 6.0*6.0*6.0, SW3 6.0*6.0*6.0, U1 STM32L431KBU6_C2826408, U10 MAX3221ECPWR, U11 HB-PH9-12727PB2GOB, X1 SC-32S32.768kHz20PPM7pF

Commit message: pre placement and type c routing
Connections:
- net RGB_LEDS_R: no longer R33.2
- net SWCLK: now also R41.1
- net SWDIO: no longer R41.1
- new net RGB_LEDS: R33.2
Other:
- note removed: "VBAT"
- moved on the sheet: R41
Changed lines of the file:
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@@
 	(text "VDD"
 		(exclude_from_sim no)
-		(at 42.164 24.384 0)
+		(at 51.054 24.638 0)
 		(effects
 			(font
@@
 		)
 	)
-	(text "VDDA"
+	(text "VDD"
 		(exclude_from_sim no)
-		(at 59.436 24.638 0)
+		(at 67.31 24.892 0)
 		(effects
 			(font
@@
 		)
 	)
-	(text "Original part number for the stm32 v3 set is :\nFTSH-107-01-L-DV-K-A\n"
+	(text "VDDA"
 		(exclude_from_sim no)
-		(at 338.328 208.28 0)
+		(at 59.436 24.638 0)
 		(effects
 			(font
 				(size 1.27 1.27)
-				(thickness 0.254)
-				(bold yes)
 			)
 		)
 	)
-	(text "VBAT"
+	(text "Original part number for the stm32 v3 set is :\nFTSH-107-01-L-DV-K-A\n"
 		(exclude_from_sim no)
-		(at 67.564 24.638 0)
+		(at 338.328 208.28 0)
 		(effects
 			(font
 				(size 1.27 1.27)
+				(thickness 0.254)
+				(bold yes)
 			)
 		)
@@
 	(text "VDDA"
 		(exclude_from_sim no)
-		(at 50.8 24.638 0)
+		(at 42.164 24.638 0)
 		(effects
 			(font
@@
 	(wire
 		(pts
+			(xy 300.99 223.52) (xy 331.47 223.52)
+		)
+		(stroke
+			(width 0)
+			(type default)
+		)
+	)
+	(wire
+		(pts
 			(xy 50.8 41.91) (xy 41.91 41.91)
 		)
@@
 	(wire
 		(pts
-			(xy 308.61 220.98) (xy 308.61 227.33)
-		)
-		(stroke
-			(width 0)
-			(type default)
-		)
-	)
-	(wire
-		(pts
 			(xy 50.8 39.37) (xy 50.8 41.91)
 		)
@@
 	(wire
 		(pts
-			(xy 300.99 223.52) (xy 331.47 223.52)
-		)
-		(stroke
-			(width 0)
-			(type default)
-		)
-	)
-	(wire
-		(pts
 			(xy 350.52 233.68) (xy 350.52 237.49)
 		)
@@
 	(wire
 		(pts
-			(xy 308.61 237.49) (xy 308.61 240.03)
+			(xy 300.99 236.22) (xy 300.99 238.76)
 		)
 		(stroke
@@
 	(wire
 		(pts
+			(xy 300.99 223.52) (xy 300.99 226.06)
+		)
+		(stroke
+			(width 0)
+			(type default)
+		)
+	)
+	(wire
+		(pts
 			(xy 50.8 26.67) (xy 50.8 29.21)
 		)
@@
 		)
 	)
-	(hierarchical_label "RGB_LEDS_R"
+	(hierarchical_label "RGB_LEDS"
 		(shape output)
 		(at 290.83 71.12 0)
@@
 	(symbol
 		(lib_id "power:GND")
-		(at 308.61 240.03 0)
+		(at 300.99 238.76 0)
 		(mirror y)
 		(unit 1)
@@
 		(dnp no)
 		(property "Reference" "#PWR019"
-			(at 308.61 246.38 0)
+			(at 300.99 245.11 0)
 			(effects
 				(font
@@
 		)
 		(property "Value" "GND"
-			(at 308.61 243.84 0)
+			(at 300.99 242.57 0)
 			(effects
 				(font
@@
 		)
 		(property "Footprint" ""
-			(at 308.61 240.03 0)
+			(at 300.99 238.76 0)
 			(effects
 				(font
@@
 		)
 		(property "Datasheet" ""
-			(at 308.61 240.03 0)
+			(at 300.99 238.76 0)
 			(effects
 				(font
@@
 		)
 		(property "Description" "Power symbol creates a global label with name \"GND\" , ground"
-			(at 308.61 240.03 0)
+			(at 300.99 238.76 0)
 			(effects
 				(font
@@
 	(symbol
 		(lib_id "easyeda2kicad:0603WAF1001T5E")
-		(at 308.61 232.41 270)
+		(at 300.99 231.14 270)
 		(unit 1)
 		(exclude_from_sim yes)
@@
 		(dnp yes)
 		(property "Reference" "R41"
-			(at 309.88 231.14 90)
+			(at 302.26 229.87 90)
 			(effects
 				(font
@@
 		)
 		(property "Value" "0603WAF1001T5E"
-			(at 303.53 232.41 0)
+			(at 295.91 231.14 0)
 			(effects
 				(font
@@
 		)
 		(property "Footprint" "easyeda2kicad:R0603"
-			(at 300.99 232.41 0)
+			(at 293.37 231.14 0)
 			(effects
 				(font
@@
 		)
 		(property "Datasheet" "https://lcsc.com/product-detail/Chip-Resistor-Surface-Mount-UniOhm_1KR-1001-1_C21190.html"
-			(at 298.45 232.41 0)
+			(at 290.83 231.14 0)
 			(effects
 				(font
@@
 		)
 		(property "Description" "1K"
-			(at 309.88 233.68 90)
+			(at 302.26 232.41 90)
 			(effects
 				(font
@@
 		)
 		(property "LCSC Part" "C21190"
-			(at 295.91 232.41 0)
+			(at 288.29 231.14 0)
 			(effects
 				(font
