File: stm32.kicad_sch (KiCad schematic)
At the start: 0 parts

Commit message: all done except rgb leds and i2c sns
Other:
- sheet stm32_page ports: added RGB_LEDS; removed RGB_LEDS_R
Changed lines of the file:
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@@
-			)
-		)
-		(pin "RGB_LEDS_R" output
-			(at 157.48 43.18 0)
-			(effects
-				(font
-					(size 1.27 1.27)
-				)
-				(justify right)
 			)
 		)
@@
 			)
 		)
+		(pin "RGB_LEDS" output
+			(at 157.48 43.18 0)
+			(effects
+				(font
+					(size 1.27 1.27)
+				)
+				(justify right)
+			)
+		)
