File: usb_power.kicad_sch (KiCad schematic)
At the start: 48 parts, among them CN1 SM04B-SRSS-TB (LF)(SN), J3 B2B-PH-SM4-TB (LF)(SN), P1 TYPE-C 16PIN 2MD(073), Q1 DMG2301L-7, SW1 JS102011JCQN, U13 CH340C_C7464026, U2 MCP73833T-AMI/MF, U3 TPS631000DRLR, U5 XC6206P332MR_C347376, U6 INA260AIPWR

Commit message: pre placement and type c routing
Connections:
- net +5V: now also U5.3 (VIN), U6.14 (IN-), U6.15 (IN-), U6.16 (IN-); no longer C1.2, C133.2, C134.2, R1.2, U3.1 (VOUT), U6.1 (IN+), U6.10 (VS), U6.12 (VBUS), U6.2 (IN+), U6.3 (IN+)
- new net 5V_INA: C1.2, C133.2, C134.2, R1.2, U3.1 (VOUT), U6.1 (IN+), U6.10 (VS), U6.12 (VBUS), U6.2 (IN+), U6.3 (IN+)
Changed lines of the file:
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@@
 	)
 	(junction
-		(at 358.775 133.35)
-		(diameter 0)
-		(color 0 0 0 0)
-	)
-	(junction
 		(at 373.38 201.93)
 		(diameter 0)
@@
 	(wire
 		(pts
-			(xy 358.775 129.54) (xy 358.775 133.35)
-		)
-		(stroke
-			(width 0)
-			(type default)
-		)
-	)
-	(wire
-		(pts
 			(xy 278.13 72.39) (xy 278.13 93.98)
 		)
@@
 	(wire
 		(pts
-			(xy 358.775 133.35) (xy 367.03 133.35)
+			(xy 350.52 133.35) (xy 367.03 133.35)
 		)
 		(stroke
@@
 	(wire
 		(pts
-			(xy 350.52 133.35) (xy 358.775 133.35)
-		)
-		(stroke
-			(width 0)
-			(type default)
-		)
-	)
-	(wire
-		(pts
 			(xy 238.76 124.46) (xy 247.65 124.46)
 		)
@@
 	(wire
 		(pts
+			(xy 330.2 185.42) (xy 330.2 189.23)
+		)
+		(stroke
+			(width 0)
+			(type default)
+		)
+	)
+	(wire
+		(pts
 			(xy 53.34 243.84) (xy 53.34 229.87)
 		)
@@
 			"////////////////////////////////////////////mZmZmZmZmZmZmZmZmZmZmZmZmZmZmZmZ"
 			"mZmZmZmZmZmZmZmZmZmZmZmZmZmZmZmZmZmZmZmZmZmZmZmZmZmZmZmZmZmZmZmZmZmZmZmZmZmZ"
-			"mZmZmQ=="
+			"mZmZmQAAAAAAAAAAAAAAAAAAAAAAAAAAAAAAAAAAAAAAAAAAAAAAAAAAAAAAAAAAAAAAAAAAAAAA"
+			"AAAAAAAAAAAAAAAAAAAAAAAAAAAAAAAAAAAAAAAAAAAAAAAAAAAAAAAAAAAAAAAAAAAAAAAAAAAA"
+			"AAAAAAAAAAAAAAAAAAAAAAAAAAAAAAAAAAAAAAAAAAAAAAAAAAAAAAAAAAAAAAAAAAAAAAAAAAAA"
+			"AAAAAAAAAAAAAAAAAAAAAAAAAAAAAAAAAAAAAAAAAAAAAAAAAAAAAAAAAAAAAAAAAAAAAAAAAAAA"
+			"AAAAAAAAAAAAAAAAAAAAAAAAAAAAAAAAAAAAAAAAAAAAAAAAAAAAAAAAAAAAAAAAAAAAAAAAAAAA"
+			"AAAAAAAAAAAAAAAAAAAAAAAAAAAAAAAAAAAAAAAAAAAAAAAAAAAAAAAAAAAAAAAAAAAAAAAAAAAA"
+			"AAAAAAAAAAAAAAAAAAAAAAAAAAAAAAAAAAAAAAAAAAAAAAAAAAAAAAAAAAAAAAAAAAAAAAAAAAAA"
+			"AAAAAAAAAAAAAAAAAAAAAAAAAAAAAAAAAAAAAAAAAAAAAAAAAAAAAAAAAAAAAAAAAAAAAAAAAAAA"
+			"AAAAAAAAAAAAAAAAAAAAAAAAAAAAAAAAAAAAAAAAAAAAAAAAAAAAAAAAAAAAAAAAAAAAAAAAAAAA"
+			"AAAAAAAAAAAAAAAAAAAAAAAAAAAAAAAAAAAAAAAAAAAAAAAAAAAAAAAAAAAAAAAAAAAAAAAAAAAA"
+			"AAAAAAAAAAAAAAAAAAAAAAAAAAAAAAAAAAAAAAAAAAAAAAAAAAAAAAAAAAAAAAAAAAAAAAAAAAAA"
+			"AAAAAAAAAAAAAAAAAAAAAAAAAAAAAAAAAAAAAAAAAAAAAAAAAAAAAAAAAAAAAAAAAAAAAAAAAAAA"
+			"AAAAAAAAAAAAAAAAAAAAAAAAAAAAAAAAAAAAAAAAAAAAAAAAAAAAAAAAAAAAAAAAAAAAAAAAAAAA"
+			"AAAAAAAAAAAAAAAAAAAAAAAAAAAAAAAAAAAAAAAAAAAAAAAAAAAAAAAAAAAAAAAAAAAAAAAAAAAA"
+			"AAAAAAAAAAAAAAAAAAAAAAAAAAAAAAAAAAAAAAAAAAAAAAAAAAAAAAAAAAAAAAAAAAAAAAAAAAAA"
+			"AAAAAAAAAAAAAAAAAAAAAAAAAAAAAAAAAAAAAAAAAAAAAAAAAAAAAAAAAAAAAAAAAAAAAAAAAAAA"
+			"AAAAAAAAAAAAAAAAAAAAAAAAAAAAAAAAAAAAAAAAAAAAAAAAAAAAAAAAAAAAAAAAAAAAAAAAAAAA"
+			"AAAAAAAAAAAAAAAAAAAAAAAAAAAAAAAAAAAAAAAAAAAAAAAAAAAAAAAAAAAAAAAAAAAAAAAAAAAA"
+			"AAAAAA=="
 		)
 	)
@@
 			"AAB/9Z2eAFIHgPzBLUFIIK7BhHjZPUGFLkFGIK7BU0EuPgAAAAAAAAAAAAAAAAAAAAAAAAAA/+gE"
 			"AAEAAAAAAAAAQ/WhngBTB4CjSjJBedCwwVFBLj7eZDJBGUmwwfe+3D6wXBC87AEAAHBWELzsAQAA"
-			"AQAAAAAAAAAAAAAAAAAAAEf1pZ4AVAeAo0oyQbJPsMFRQS4+3mQyQQ=="
+			"AQAAAAAAAAAAAAAAAAAAAEf1pZ4AVAeAo0oyQbJPsMFRQS4+3mQyQXQAdABPAFgAbABaAFUAUgAv"
+			"AFkASgBmAFEANgBWAFMAYQBWAGwAcABHAFEASQBvAEsAUwBuAGgAagBnAHAAdgAzAGIAcgBWAHcA"
+			"cwB3AEMASQB4AHcAWgBHAFgAbgB4ADQAawBYACsARQAvAGYAcwAyAFkATQBBACsASABYAGYAdwBN"
+			"AEQAQQAxAHQAWQBXAEEAYwA3AE0AegBDAFMAYQBTAEcAaABvAEsAUABGAHQAVgBsAEoAYQBBAGcA"
+			"QwBBAG8AYQBTADQAaABKADkASQBjAFgARQB4ADYAWAA5AEwAVwBIAE4AOQA4ACsAZgBQAEoAeQBh"
+			"ADcAeQBzAHYATABoAHcANABkAHUAbQB6AFoAcwBnAHMAWABMAHQAeQA3AGQAMgAvAG4AegBwADMA"
+			"awBvADIAegBmAHYAbwAwAHQASQBuAEsASQBBADYAdABxAFYARgArAEEAcAByAFYAcwBWAFQAOABK"
+			"AFEAcQBGAFEAbQBDAEEAVQB4AHAAUAAvAEMATwBPAEYAUQBxAEYAUQBHAEoAOABnAFQAQgBBAEsA"
+			"aABVAEkAZgBIAHgAOQA1AHoANwBzADgAYwBuAEoAeQAvAHYAMwAzAFgAOQBhAFYAYwAyADMARwBE"
+			"AFEAMABOAFEAMABOAEQASAB6ADUAOABXAEYAWgBXAHgAawBWAE8AUwBrAG8AYQBOAG0AdwBZAEcA"
+			"dwBVAEIAQQBnADgAUABqACsAagBvAGEASwBsAFUAKwB1AGUAZgBmADMASwBlAG8AOABtAC8AMwAz"
+			"ADMAMwBYAFgAbAA1AGUAWABKAHkAOABzAGgAUABSAGsATAB0AFAAZgBEAEIAQgB4ADgAawBKAEMA"
+			"UwBVAGwAcABZAEcAQgBRAFgAeABIAG8AcgBzADcAZQAyAHYAWABiAHQARwBIAEIALwBmAHUAMwBm"
+			"AFAAeABNAFIAVQBhAFQARgAyAGQAdQAyAGMAbgA1ACsAUABNAFUANQBMAFMANQBzADkAZQB6AFkA"
+			"LwBqAG8AbQBwAHkAZABHAGoAUgA3AE8AegBzADkAVwA4AEwAeQBFADUATwBmAG4ASQBrAFMATwA5"
+			"AGUAdgBlAFMAVAA3AHgAegA1AC8AMABIADkAdAArADgAZQBWAE8AVgBNADMAcQB1AG8AUABpAGwA"
+			"MQBiAEoAbABTADMAdgA3AFYAdgB3AGcATABTADIAdAAvAC8ANgA3AGkAVABGACsAOABPAEMAQgB2"
+			"AEkAawA4AHgATAArAFYAKwBhAEcAcgBxAHoAdAAvAC8AdgB6AG4AegA1ADgAVABCAFoANgA3ADUA"
+			"dQBuAHAAZQBlAC8AZQBQAGYASgBvAGMAaQBRAEoAOABSAE4AQwBzAA=="
+		)
+	)
+	(label "5V_INA"
+		(at 368.3 133.35 0)
+		(effects
+			(font
+				(size 1.27 1.27)
+			)
+			(justify left bottom)
 		)
 	)
@@
 		(length 2.54)
 		(shape round)
+		(at 294.64 189.23 0)
+		(fields_autoplaced yes)
+		(effects
+			(font
+				(size 1.27 1.27)
+			)
+			(justify left bottom)
+		)
+		(property "Netclass" "power"
+			(at 295.3385 186.69 0)
+			(effects
+				(font
+					(size 1.27 1.27)
+					(italic yes)
+				)
+				(justify left)
+			)
+		)
+	)
+	(netclass_flag ""
+		(length 2.54)
+		(shape round)
 		(at 264.16 72.39 0)
 		(fields_autoplaced yes)
@@
 		(lib_name "+5V_1")
 		(lib_id "power:+5V")
-		(at 358.775 129.54 0)
+		(at 330.2 185.42 0)
 		(unit 1)
 		(exclude_from_sim no)
@@
 		(fields_autoplaced yes)
 		(property "Reference" "#PWR0210"
-			(at 358.775 133.35 0)
+			(at 330.2 189.23 0)
 			(effects
 				(font
@@
 		)
 		(property "Value" "+5V"
-			(at 358.775 125.095 0)
+			(at 330.2 180.975 0)
 			(effects
 				(font
@@
 		)
 		(property "Footprint" ""
-			(at 358.775 129.54 0)
+			(at 330.2 185.42 0)
 			(effects
 				(font
@@
 		)
 		(property "Datasheet" ""
-			(at 358.775 129.54 0)
+			(at 330.2 185.42 0)
 			(effects
 				(font
@@
 		)
 		(property "Description" "Power symbol creates a global label with name \"+5V\""
-			(at 358.775 129.54 0)
+			(at 330.2 185.42 0)
 			(effects
 				(font

Commit message: routing all power
Parts:
- added C8: CC0603KRX7R9BB104, easyeda2kicad:C0603, symbol easyeda2kicad:CC0603KRX7R9BB104
Connections:
- net 5V_INA: now also C8.2
- net GND: now also C8.1
Other:
- moved on the sheet: R43
Changed lines of the file:
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@@
 	(wire
 		(pts
+			(xy 386.08 185.42) (xy 386.08 186.69)
+		)
+		(stroke
+			(width 0)
+			(type default)
+		)
+	)
+	(wire
+		(pts
 			(xy 350.52 153.67) (xy 350.52 159.385)
 		)
@@
 	(wire
 		(pts
+			(xy 386.08 172.72) (xy 375.92 172.72)
+		)
+		(stroke
+			(width 0)
+			(type default)
+		)
+	)
+	(wire
+		(pts
 			(xy 314.96 204.47) (xy 314.96 172.72)
 		)
@@
 	(wire
 		(pts
+			(xy 386.08 175.26) (xy 386.08 172.72)
+		)
+		(stroke
+			(width 0)
+			(type default)
+		)
+	)
+	(wire
+		(pts
 			(xy 68.58 163.83) (xy 68.58 170.18)
 		)
@@
 	(wire
 		(pts
-			(xy 330.2 189.23) (xy 257.81 189.23)
+			(xy 257.81 189.23) (xy 330.2 189.23)
 		)
 		(stroke
@@
 			"AAAAAAAAAAAAAAAAAAAAAAAAAAAAAAAAAAAAAAAAAAAAAAAAAAAAAAAAAAAAAAAAAAAAAAAAAAAA"
 			"AAAAAAAAAAAAAAAAAAAAAAAAAAAAAAAAAAAAAAAAAAAAAAAAAAAAAAAAAAAAAAAAAAAAAAAAAAAA"
+			"AAAAAAAAAAAAAAAAAAAAAAAAAAAAAAAAAAAAAAAAAAAAAAAAAAAAAAAAAAAAAAAAAAAAAAAAAAAA"
+			"AAAAAAAAAAAAAAAAAAAAAAAAAAAAAAAAAAAAAAAAAAAAAAAAAAAAAAAAAAAAAAAAAAAAAAAAAAAA"
+			"AAAAAAAAAAAAAAAAAAAAAAAAAAAAAAAAAAAAAAAAAAAAAAAAAAAAAAAAAAAAAAAAAAAAAAAAAAAA"
+			"AAAAAAAAAAAAAAAAAAAAAAAAAAAAAAAAAAAAAAAAAAAAAAAAAAAAAAAAAAAAAAAAAAAAAAAAAAAA"
+			"AAAAAAAAAAAAAAAAAAAAAAAAAAAAAAAAAAAAAAAAAAAAAAAAAAAAAAAAAAAAAAAAAAAAAAAAAAAA"
+			"AAAAAAAAAAAAAAAAAAAAAAAAAAAAAAAAAAAAAAAAAAAAAAAAAAAAAAAAAAAAAAAAAAAAAAAAAAAA"
+			"AAAAAAAAAAAAAAAAAAAAAAAAAAAAAAAAAAAAAAAAAAAAAAAAAAAAAAAAAAAAAAAAAAAAAAAAAAAA"
+			"AAAAAAAAAAAAAAAAAAAAAAAAAAAAAAAAAAAAAAAAAAAAAAAAAAAAAAAAAAAAAAAAAAAAAAAAAAAA"
+			"AAAAAAAAAAAAAAAAAAAAAAAAAAAAAAAAAAAAAAAAAAAAAAAAAAAAAAAAAAAAAAAAAAAAAAAAAAAA"
+			"AAAAAAAAAAAAAAAAAAAAAAAAAAAAAAAAAAAAAAAAAAAAAAAAAAAAAAAAAAAAAAAAAAAAAAAAAAAA"
+			"AAAAAAAAAAAAAAAAAAAAAAAAAAAAAAAAAAAAAAAAAAAAAAAAAAAAAAAAAAAAAAAAAAAAAAAAAAAA"
+			"AAAAAAAAAAAAAAAAAAAAAAAAAAAAAAAAAAAAAAAAAAAAAAAAAAAAAAAAAAAAAAAAAAAAAAAAAAAA"
+			"AAAAAAAAAAAAAAAAAAAAAAAAAAAAAAAAAAAAAAAAAAAAAAAAAAAAAAAAAAAAAAAAAAAAAAAAAAAA"
+			"AAAAAAAAAAAAAAAAAAAAAAAAAAAAAAAAAAAAAAAAAAAAAAAAAAAAAAAAAAAAAAAAAAAAAAAAAAAA"
+			"AAAAAAAAAAAAAAAAAAAAAAAAAAAAAAAAAAAAAAAAAAAAAAAAAAAAAAAAAAAAAAAAAAAAAAAAAAAA"
+			"AAAAAAAAAAAAAAAAAAAAAAAAAAAAAAAAAAAAAAAAAAAAAAAAAAAAAAAAAAAAAAAAAAAAAAAAAAAA"
+			"AAAAAAAAAAAAAAAAAAAAAAAAAAAAAAAAAAAAAAAAAAAAAAAAAAAAAAAAAAAAAAAAAAAAAAAAAAAA"
+			"AAAAAAAAAAAAAAAAAAAAAAAAAAAAAAAAAAAAAAAAAAAAAAAAAAAAAAAAAAAAAAAAAAAAAAAAAAAA"
 			"AAAAAA=="
 		)
@@
 			"MQBiAEoAbABTADMAdgA3AFYAdgB3AGcATABTADIAdAAvAC8ANgA3AGkAVABGACsAOABPAEMAQgB2"
 			"AEkAawA4AHgATAArAFYAKwBhAEcAcgBxAHoAdAAvAC8AdgB6AG4AegA1ADgAVABCAFoANgA3ADUA"
-			"dQBuAHAAZQBlAC8AZQBQAGYASgBvAGMAaQBRAEoAOABSAE4AQwBzAA=="
+			"dQBuAHAAZQBlAC8AZQBQAGYASgBvAGMAaQBRAEoAOABSAE4AQwBzAHUAYgBDAGkAUwBNAFoAQgBH"
+			"AEIAZwBZAFAARABEAEQAegAvAGMAdgBSAHMAVgBHAFIAbABKAHgAaQBSADkAKwB2AFQAaAAxAHkA"
+			"TwBwAFYARAByAHYALwB4AGgALwBzAHgAWQBXAEYAdQBuAHAANgBTAFMAOABvAHEASgBpADkATwBq"
+			"AFIASgBOAHoAQQB3AE8ARAArAC8AZgB0AHkALwBjAEwAeAA0ADgAZAA1AGIAaABSAHIAOAA2ACsA"
+			"dgByADMALwAyADcARgBrAHUAMgB0AFcAcgBWADAAMwBOAHUASgAzADUAMABMAEYAVAB4AHoAWgB0"
+			"ADIAcwBoADkAWAAyAE4AagA0AHoATgBuAHoAcQBnAHAAdQBsAE8AbgBUAHAAbQBZAG0AaQBpAHAA"
+			"UgBBAGoAcwA3AE8AegArAHUALwBrAGYARgAvAFAAYQB0AFcAdgBjAGYAZwAxAC8AZgAvACsARwBk"
+			"AEQAcAAzADcAdAB4AEIAUwBDAEIAWAAvAG4ANQArAGYAbgBaADIAZABpAFIAUQBUADEALwBQADAA"
+			"ZABFAFIAWQAvAHoAdwA0AFUATQA5AGYAZQBhAFYAbAB5ADUAZABLAGwAOQBEAEEAUQBEAGcAMgBM"
+			"AEYAagBkAGIASgB0AHcAbQBUADcAeQBwAFUAcgBKAE4AdQA3AGQAdQAwAEMAQQBGAHQAYgBXADMA"
+			"NwBkAHgAeABnAFAASABqAHkAWQBwAEcARgBsAFoAZABXADEAYQAxAGMANwBPADcAdQBZAG0ASgBp"
+			"AHkAcwBqAEwARwBsAEQAUwBnAFEAWQBNAEcAOABXAHYASwBnAEEARQBEAHkAQwBPADcAZAArACsA"
+			"ZQBuAHAANQBCAHcAaQBNAGoASQAvAFgAMQA5AFcAdABmAGcAMgAwAGYAOQBQAFQAMAB1AEkAOQBT"
+			"AFgAbAA1AE8AdgBpAHgAUwA4AFcAVgBmAGoAUABEAEQAUwBzAFQANwAxAFEARwBjAGIAawB2AFUA"
+			"VwArAFkASABHAHoASgBJAHIAYQBMAEwATwBoACsAWAAzADIAUABCAC8AWABuAGcAdwBBAEUAdQA4"
+			"AG0AZQBmAGYAVgBaAFgAMAB3AEkAQQA2AE4AVwB6ADUANgBOAEgAagA1AEQAOAB2AFEAZwBBAGoA"
+			"aAA4AC8AegB0AGEAYwBPAHUAbABQAG4ARABoAHgAdgA4AEkATwBmAGcAQgBBAEMAQgBVAFcARgBw"
+			"AEoAbgBwAGEAVwBsAGsAWgBhAGQAYQA5AGoAMQA5AGYAWAA5AC8AZgAyAEoASQAxAE8ATQA4AFkA"
+			"dwBaAE0ALwBoADUANABYADUALwAvAFAASABIADkAUgBiAFoAMgBMAA=="
 		)
 	)
@@
 	)
 	(symbol
+		(lib_id "easyeda2kicad:CC0603KRX7R9BB104")
+		(at 386.08 180.34 90)
+		(unit 1)
+		(exclude_from_sim no)
+		(in_bom yes)
+		(on_board yes)
+		(dnp no)
+		(property "Reference" "C8"
+			(at 388.112 176.276 90)
+			(effects
+				(font
+					(size 1.27 1.27)
+				)
+				(justify right)
+			)
+		)
+		(property "Value" "CC0603KRX7R9BB104"
+			(at 389.89 181.6099 90)
+			(effects
+				(font
+					(size 1.27 1.27)
+				)
+				(justify right)
+				(hide yes)
+			)
+		)
+		(property "Footprint" "easyeda2kicad:C0603"
+			(at 393.7 180.34 0)
+			(effects
+				(font
+					(size 1.27 1.27)
+				)
+				(hide yes)
+			)
+		)
+		(property "Datasheet" "https://lcsc.com/product-detail/Multilayer-Ceramic-Capacitors-MLCC-SMD-SMT_100nF-104-10-50V_C14663.html"
+			(at 396.24 180.34 0)
+			(effects
+				(font
+					(size 1.27 1.27)
+				)
+				(hide yes)
+			)
+		)
+		(property "Description" "100nF"
+			(at 390.144 178.054 90)
+			(effects
+				(font
+					(size 1.27 1.27)
+				)
+			)
+		)
+		(property "LCSC Part" "C14663"
+			(at 398.78 180.34 0)
+			(effects
+				(font
+					(size 1.27 1.27)
+				)
+				(hide yes)
+			)
+		)
+		(property "Field6" "0603"
+			(at 386.08 180.34 90)
+			(effects
+				(font
+					(size 0.635 0.635)
+				)
+			)
+		)
+		(pin "1"
+		)
+		(pin "2"
+		)
+		(instances
+			(project "stm32"
+				(path "/6657db5f-e034-448d-bae3-f44b9f033a3a/6f1f01ea-fc88-494c-8e17-b18350ce0e3a"
+					(reference "C8")
+					(unit 1)
+				)
+			)
+		)
+	)
+	(symbol
 		(lib_id "easyeda2kicad:0603WAF8060T5E")
 		(at 328.93 140.97 270)
@@
 	)
 	(symbol
+		(lib_id "SAMC21_breakout-rescue:GND")
+		(at 386.08 186.69 0)
+		(unit 1)
+		(exclude_from_sim no)
+		(in_bom yes)
+		(on_board yes)
+		(dnp no)
+		(property "Reference" "#PWR0425"
+			(at 386.08 193.04 0)
+			(effects
+				(font
+					(size 1.27 1.27)
+				)
+				(hide yes)
+			)
+		)
+		(property "Value" "GND"
+			(at 386.08 190.5 0)
+			(effects
+				(font
+					(size 1.27 1.27)
+				)
+			)
+		)
+		(property "Footprint" ""
+			(at 386.08 186.69 0)
+			(effects
+				(font
+					(size 1.27 1.27)
+				)
+			)
+		)
+		(property "Datasheet" ""
+			(at 386.08 186.69 0)
+			(effects
+				(font
+					(size 1.27 1.27)
+				)
+			)
+		)
+		(property "Description" ""
+			(at 386.08 186.69 0)
+			(effects
+				(font
+					(size 1.27 1.27)
+				)
+				(hide yes)
+			)
+		)
+		(pin "1"
+		)
+		(instances
+			(project "stm32"
+				(path "/6657db5f-e034-448d-bae3-f44b9f033a3a/6f1f01ea-fc88-494c-8e17-b18350ce0e3a"
+					(reference "#PWR0425")
+					(unit 1)
+				)
+			)
+		)
+	)
+	(symbol
 		(lib_id "easyeda2kicad:CC0603KRX7R9BB104")
 		(at 53.34 248.92 90)
@@
 	(symbol
 		(lib_id "easyeda2kicad:0603WAF1002T5E")
-		(at 252.73 162.56 90)
+		(at 252.73 162.56 270)
+		(mirror x)
 		(unit 1)
 		(exclude_from_sim no)
@@
 		(dnp no)
 		(property "Reference" "R43"
-			(at 255.27 161.2899 90)
+			(at 250.19 161.2899 90)
 			(effects
 				(font
@@
 		)
 		(property "Value" "0603WAF1002T5E"
-			(at 255.27 163.8299 90)
+			(at 250.19 163.8299 90)
 			(effects
 				(font
@@
 		)
 		(property "Footprint" "easyeda2kicad:R0603"
-			(at 260.35 162.56 0)
+			(at 245.11 162.56 0)
 			(effects
 				(font
@@
 		)
 		(property "Datasheet" "https://lcsc.com/product-detail/Chip-Resistor-Surface-Mount-UniOhm_10KR-1002-1_C25804.html"
-			(at 262.89 162.56 0)
+			(at 242.57 162.56 0)
 			(effects
 				(font
@@
 		)
 		(property "Description" "10k"
-			(at 250.698 162.56 0)
+			(at 254.762 162.56 0)
 			(effects
 				(font
@@
 		)
 		(property "LCSC Part" "C25804"
-			(at 265.43 162.56 0)
+			(at 240.03 162.56 0)
 			(effects
 				(font
